File: PCB/PCB.kicad_pcb (KiCad board)
At the start: 2 copper layers, 101.6 x 39.7 mm, 37 parts, among them J1 USB_C_Receptacle_USB2.0, SW1 SW_Push, U1 ATmega32U2-AU, Y1 16MHz

Commit message: removed silkscreen
Parts:
- removed G***: LOGO, gojo:gojo
